Commit message: autocapture to folder

File: src/alligator_sim/urdf/mybot.xacro (robot description, xacro)
@@ -139,5 +139,5 @@
   <link name="camera">
     <collision>
-      <origin xyz="0 0 0" rpy="0 0 0"/>
+      <origin xyz="0 0 0" rpy="0 0.36 0"/>
       <geometry>
         <box size="${cameraSize} ${cameraSize} ${cameraSize}"/>
@@ -145,5 +145,5 @@
     </collision>
     <visual>
-      <origin xyz="0 0 0" rpy="0 0 0"/>
+      <origin xyz="0 0 0" rpy="0 0.36 0"/>
       <geometry>
         <box size="${cameraSize} ${cameraSize} ${cameraSize}"/>
@@ -153,5 +153,5 @@
     <inertial>
       <mass value="${cameraMass}" />
-      <origin xyz="0 0 0" rpy="0 0 0"/>
+      <origin xyz="0 0 0" rpy="0 0.36 0"/>
       <box_inertia m="${cameraMass}" x="${cameraSize}" y="${cameraSize}" z="${cameraSize}" />
       <inertia ixx="1e-6" ixy="0" ixz="0" iyy="1e-6" iyz="0" izz="1e-6" />
@@ -160,16 +160,16 @@
   <joint name="camera_joint" type="fixed">
     <axis xyz="0 1 0" />
-    <origin xyz=".2 0 0" rpy="0 0 0"/>
+    <origin xyz=".2 0 0.1" rpy="0 0.36 0"/>
     <parent link="chassis"/>
     <child link="camera"/>
   </joint>
-  <joint name="hokuyo_joint" type="fixed">
+  <!-- <joint name="hokuyo_joint" type="fixed">
     <axis xyz="0 1 0" />
     <origin xyz=".15 0 .1" rpy="0 0 0"/>
     <parent link="chassis"/>
     <child link="hokuyo"/>
-  </joint>
+  </joint> -->
   <!-- Hokuyo Laser -->
-  <link name="hokuyo">
+  <!-- <link name="hokuyo">
     <collision>
       <origin xyz="0 0 0" rpy="0 0 0"/>
@@ -189,4 +189,4 @@
       <inertia ixx="1e-6" ixy="0" ixz="0" iyy="1e-6" iyz="0" izz="1e-6" />
     </inertial>
-  </link>
+  </link> -->
 </robot>
